File: hardware/leds.kicad_sch (KiCad schematic)
At the start: 28 parts, among them Q201 DMP3028, Q202 MMBT3904

Commit message: fix bom
Parts:
- R203, R204, R205, R206, R207, R208: value 50R -> 75R; LCSC ID C17470 -> C5198289
Changed lines of the file:
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@@
 			)
 		)
-		(property "Value" "50R"
+		(property "Value" "75R"
 			(at 130.81 109.2199 0)
 			(effects
@@
 			)
 		)
-		(property "LCSC ID" "C17470"
+		(property "LCSC ID" "C5198289"
 			(at 128.27 107.95 0)
 			(effects
@@
 			)
 		)
-		(property "Value" "50R"
+		(property "Value" "75R"
 			(at 146.05 109.2199 0)
 			(effects
@@
 			)
 		)
-		(property "LCSC ID" "C17470"
+		(property "LCSC ID" "C5198289"
 			(at 143.51 107.95 0)
 			(effects
@@
 			)
 		)
-		(property "Value" "50R"
+		(property "Value" "75R"
 			(at 161.29 109.2199 0)
 			(effects
@@
 			)
 		)
-		(property "LCSC ID" "C17470"
+		(property "LCSC ID" "C5198289"
 			(at 158.75 107.95 0)
 			(effects
@@
 			)
 		)
-		(property "Value" "50R"
+		(property "Value" "75R"
 			(at 190.5 109.2199 0)
 			(effects
@@
 			)
 		)
-		(property "LCSC ID" "C17470"
+		(property "LCSC ID" "C5198289"
 			(at 187.96 107.95 0)
 			(effects
@@
 			)
 		)
-		(property "Value" "50R"
+		(property "Value" "75R"
 			(at 176.53 109.2199 0)
 			(effects
@@
 			)
 		)
-		(property "LCSC ID" "C17470"
+		(property "LCSC ID" "C5198289"
 			(at 173.99 107.95 0)
 			(effects
@@
 			)
 		)
-		(property "Value" "50R"
+		(property "Value" "75R"
 			(at 205.74 109.2199 0)
 			(effects
@@
 			)
 		)
-		(property "LCSC ID" "C17470"
+		(property "LCSC ID" "C5198289"
 			(at 203.2 107.95 0)
 			(effects
