File: hardware/illuminator.kicad_pcb (KiCad board)
At the start: 4 copper layers, 85 x 100 mm, 66 parts, among them J101 HRO_TYPE_C_31_M_12, J102 PROG, J103 LCLV, Q201 DMP3028, Q202 MMBT3904, SW101 RESET, SW102 DFU, U101 SRV05-4, U102 STM32G431CBUx, U103 WAS3157B-6/TR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

Commit message: Update CI and mechanical assembly
Parts:
- SW102: footprint Button_Switch_THT:SW_Tactile_SKHH_Angled -> easyeda2kicad:KEY-TH_SKHHLWA010
- moved SW102 2.60 mm to (139.8, 144.8), turned to 0 degrees
Connections:
- SW102 pad 1: /DFU -> +3V3
- SW102 pad 2: +3V3 -> /DFU
