File: hardware/illuminator.kicad_sch (KiCad schematic)
At the start: 35 parts, among them J101 HRO_TYPE_C_31_M_12, J102 PROG, J103 LCLV, SW101 RESET, SW102 DFU, U101 SRV05-4, U102 STM32G431CBUx, U103 WAS3157B-6/TR, U104 TL072, U105 HT7550-1_C16106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

Commit message: fix erc errors
Parts:
- U103: LCSC Part (none) -> C213161
- U105: footprint Package_TO_SOT_SMD:SOT-89-3 -> easyeda2kicad:SOT-89-3_L4.5-W2.5-P1.50-LS4.2-BR; LCSC Part (none) -> C16106
- U106: footprint Package_TO_SOT_SMD:SOT-89-3 -> easyeda2kicad:SOT-89-3_L4.5-W2.5-P1.50-LS4.2-BR; LCSC Part (none) -> C71136
Connections:
- no-connect marks 3 -> 27

Commit message: heatsinking
Parts:
- J103, SW101: now left out of the parts list
Changed lines of the file:
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@@
 		(unit 1)
 		(exclude_from_sim no)
-		(in_bom yes)
+		(in_bom no)
 		(on_board yes)
 		(dnp no)
@@
 		(unit 1)
 		(exclude_from_sim no)
-		(in_bom yes)
-		(on_board yes)
-		(dnp no)
+		(in_bom no)
+		(on_board yes)
+		(dnp no)

Commit message: fix bom
Parts:
- C106, C107: LCSC ID C107145 -> C1554
Changed lines of the file:
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@@
 			)
 		)
-		(property "LCSC ID" "C107145"
+		(property "LCSC ID" "C1554"
 			(at 39.37 121.92 0)
 			(effects
@@
 			)
 		)
-		(property "LCSC ID" "C107145"
+		(property "LCSC ID" "C1554"
 			(at 59.69 121.92 0)
 			(effects

Commit message: add gain resistors
Parts:
- added R104, R105: 0R, Resistor_SMD:R_0402_1005Metric, symbol Device:R_Small_US
- U105, U106: footprint easyeda2kicad:SOT-89-3_L4.5-W2.5-P1.50-LS4.2-BR -> Package_TO_SOT_SMD:SOT-89-3
Connections:
- net at J103.1 (Pin_1), R103.1, U104.1: now also R105.2; no longer U104.2 (-)
- net at U104.3 (+): now also R104.2; no longer U103.4 (A)
- new net: R105.1, U104.2 (-)
- new net: R104.1, U103.4 (A)
Other:
- moved on the sheet: C105, U103

Commit message: fix drc
Parts:
- added R106: 10k, Resistor_SMD:R_0402_1005Metric, symbol Device:R_Small_US
Connections:
- net GND: now also U103.3 (B0), R106.2; no longer U103.1 (B1)
- net OPAMP1_VOUT: now also U103.1 (B1); no longer U103.3 (B0)
- net TIM1_CH1: now also R106.1
Changed lines of the file:
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@@
 	)
 	(junction
+		(at 177.8 115.57)
+		(diameter 0)
+		(color 0 0 0 0)
+	)
+	(junction
 		(at 267.97 133.35)
 		(diameter 0)
@@
 	)
 	(junction
+		(at 172.72 107.95)
+		(diameter 0)
+		(color 0 0 0 0)
+	)
+	(junction
 		(at 72.39 157.48)
 		(diameter 0)
@@
 	(wire
 		(pts
+			(xy 172.72 115.57) (xy 172.72 114.3)
+		)
+		(stroke
+			(width 0)
+			(type default)
+		)
+	)
+	(wire
+		(pts
+			(xy 172.72 115.57) (xy 177.8 115.57)
+		)
+		(stroke
+			(width 0)
+			(type default)
+		)
+	)
+	(wire
+		(pts
 			(xy 49.53 71.12) (xy 57.15 71.12)
 		)
@@
 	(wire
 		(pts
-			(xy 163.83 107.95) (xy 181.61 107.95)
+			(xy 163.83 107.95) (xy 172.72 107.95)
 		)
 		(stroke
@@
 	(wire
 		(pts
+			(xy 172.72 107.95) (xy 181.61 107.95)
+		)
+		(stroke
+			(width 0)
+			(type default)
+		)
+	)
+	(wire
+		(pts
 			(xy 85.09 39.37) (xy 95.25 39.37)
 		)
@@
 	(wire
 		(pts
+			(xy 172.72 107.95) (xy 172.72 109.22)
+		)
+		(stroke
+			(width 0)
+			(type default)
+		)
+	)
+	(wire
+		(pts
 			(xy 74.93 97.79) (xy 72.39 97.79)
 		)
@@
 					(unit 1)
 				)
+			)
+		)
+	)
+	(symbol
+		(lib_id "Device:R_Small_US")
+		(at 172.72 111.76 0)
+		(unit 1)
+		(exclude_from_sim no)
+		(in_bom yes)
+		(on_board yes)
+		(dnp no)
+		(property "Reference" "R106"
+			(at 170.18 110.4899 0)
+			(effects
+				(font
+					(size 1.27 1.27)
+				)
+				(justify right)
+			)
+		)
+		(property "Value" "10k"
+			(at 170.18 113.0299 0)
+			(effects
+				(font
+					(size 1.27 1.27)
+				)
+				(justify right)
+			)
+		)
+		(property "Footprint" "Resistor_SMD:R_0402_1005Metric"
+			(at 172.72 111.76 0)
+			(effects
+				(font
+					(size 1.27 1.27)
+				)
+				(hide yes)
+			)
+		)
+		(property "Datasheet" "~"
+			(at 172.72 111.76 0)
+			(effects
+				(font
+					(size 1.27 1.27)
+				)
+				(hide yes)
+			)
+		)
+		(property "Description" "Resistor, small US symbol"
+			(at 172.72 111.76 0)
+			(effects
+				(font
+					(size 1.27 1.27)
+				)
+				(hide yes)
+			)
+		)
+		(property "LCSC ID" "C25744"
+			(at 172.72 111.76 0)
+			(effects
+				(font
+					(size 1.27 1.27)
+				)
+				(hide yes)
+			)
+		)
+		(pin "2"
+		)
+		(pin "1"
+		)
+		(instances
+			(project "illuminator"
+				(path "/acb50d16-19ca-41e0-a3c9-c32dd495407e"
+					(reference "R106")
+					(unit 1)
+				)

Commit message: Update CI and mechanical assembly
Parts:
- SW102: footprint Button_Switch_THT:SW_Tactile_SKHH_Angled -> easyeda2kicad:KEY-TH_SKHHLWA010
Connections:
- net +3V3: now also SW102.1; no longer SW102.2
- net DFU: now also SW102.2; no longer SW102.1
Changed lines of the file:
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@@
 		(lib_id "Switch:SW_Push")
 		(at 80.01 97.79 0)
-		(mirror y)
 		(unit 1)
 		(exclude_from_sim no)
@@
 			)
 		)
-		(property "Footprint" "Button_Switch_THT:SW_Tactile_SKHH_Angled"
+		(property "Footprint" "easyeda2kicad:KEY-TH_SKHHLWA010"
 			(at 80.01 92.71 0)
 			(effects
